File: boards/RC107_ROM_RAM_Board/RC107-68000_ROM_RAM_1.kicad_sch (KiCad schematic)
At the start: 26 parts, among them J1 RCBus_80PIN_68000, J10 Conn_01x06, J11 Conn_01x06, J12 Conn_01x06, J2 Conn_01x03, J3 Conn_01x03, J4 Conn_01x03, J5 Conn_01x03, J6 Conn_01x03, J7 Conn_01x03, J8 Conn_01x03, J9 Conn_01x03, U1 74LS125, U2 74LS139, U3 SST39SF040, U4 SST39SF040, U5 74LS138, U6 AS6C4008-55PCN, U7 AS6C4008-55PCN

Commit message: Updated RC107
Parts:
- added JP1, JP2: SolderJumper_2_Open, Jumper:SolderJumper-2_P1.3mm_Open_Pad1.0x1.5mm, symbol Jumper:SolderJumper_2_Open
- added R1, R2: 10K, Resistor_THT:R_Axial_DIN0207_L6.3mm_D2.5mm_P7.62mm_Horizontal, symbol Device:R
Connections:
- net ~{RAM_CS} is gone; now on net ~{CS_BANK0}: U1.1
- net ~{ROM_CS} is gone; now on net ~{CS_BANK1}: U1.4
- net +5V: now also R1.1, R2.1
- net ~{CS_BANK0}: now also JP1.2 (B), R1.2
- net ~{CS_BANK1}: now also JP2.2 (B), R2.2
- net ~{CS_ROM}: now reaches J1.45 (~{CS0})
- net ~{CS_ROM}: now also JP1.1 (A)
- net ~{CS_RAM}: now reaches J1.46 (~{CS1})
- net ~{CS_RAM}: now also JP2.1 (A)
- no-connect marks 40 -> 38
Other:
- note added: "NOTE: THE ~{CS_BANK0} AND ~{CS_BANK1} SIGNALS CAN BE SUPPLIED FROM THE MC68302 PROCESSOR ~{CS0} AND ~{CS1} PINS - CALLED ~{CS_ROM} AND ~{CS_RAM} ON THE MC68302 SCHEMATIC. IF USING THE MC68302 BOARD, THEN U1 AND U5 CAN BE OMITTED. INSTEAD, MAKE SOLDER JUMPERS JP1 & JP2 AND FIT THE BOOT ROMS INTO BANK 0 AND RAMS INTO BANK 1."
- note removed: "*~{CS_BANK0}"
- note removed: "*~{CS_BANK1}"
- note removed: "NOTE: THE ~{CS_BANK0} AND ~{CS_BANK1} SIGNALS CAN BE SUPPLIED FROM THE MC68302 PROCESSOR ~{CS0} AND ~{CS1} PINS - CALLED ~{CS_ROM} AND ~{CS_RAM} ON THE MC68302 SCHEMATIC. IF USING THE MC68302 BOARD, THEN U1 AND U5 CAN BE OMITTED. INSTEAD, CONNECT A WIRE LINK FROM J1-45 TO J11 AND A WIRE LINK FROM J1-46 TO J12 AND FIT THE BOOT ROMS INTO BANK 0."
- title: (none) -> RCBus-68K ROM / RAM Board v2
- moved on the sheet: J12
